Commit message: keep gazebo param for legacy reason
Signed-off-by: Alejandro Hernandez Cordero <ahcorde@gmail.com>

File: irobot_create_common/irobot_create_description/urdf/bumper.urdf.xacro (robot description, xacro)
@@ -13,5 +13,5 @@
   <link name="${link_name}"/>
 </xacro:macro>
-<xacro:macro name="bumper" params="name:=bumper namespace parent_link:=base_link update_rate:=62.0 visual_mesh collision_mesh
+<xacro:macro name="bumper" params="name:=bumper namespace parent_link:=base_link update_rate:=62.0 gazebo:=ignition visual_mesh collision_mesh
   *origin *inertial">
   <xacro:property name="link_name" value="${name}"/>

File: irobot_create_common/irobot_create_description/urdf/common_properties.urdf.xacro (robot description, xacro)
@@ -45,5 +45,5 @@
             h_samples h_res h_min_angle h_max_angle
             v_samples:=1 v_res:=1 v_min_angle:=0 v_max_angle:=0
-            r_min r_max r_res">
+            r_min r_max r_res gazebo:=ignition">
     <sensor name="${sensor_name}" type="gpu_lidar">
       <update_rate>${update_rate}</update_rate>

File: irobot_create_common/irobot_create_description/urdf/create3.urdf.xacro (robot description, xacro)
@@ -11,4 +11,6 @@
   <xacro:include filename="$(find irobot_create_description)/urdf/sensors/optical_mouse.urdf.xacro"/>
   <xacro:include filename="$(find irobot_create_description)/urdf/wheel_with_wheeldrop.urdf.xacro" />
+  <!-- Gazebo version (kept for legacy reasons) -->
+  <xacro:arg name="gazebo"                       default="ignition" />
   <!-- Namespace -->
   <xacro:arg name="namespace"                    default=""/>
@@ -60,4 +62,5 @@
   <!-- Bumper -->
   <xacro:bumper
+      gazebo="$(arg gazebo)"
       namespace="$(arg namespace)"
       visual_mesh="package://irobot_create_description/meshes/bumper_visual.dae"
@@ -72,8 +75,8 @@
   </xacro:bumper>
   <!-- Wheels with mechanical wheel drop -->
-  <xacro:wheel_with_wheeldrop name="left" namespace="$(arg namespace)">
+  <xacro:wheel_with_wheeldrop name="left" gazebo="$(arg gazebo)" namespace="$(arg namespace)">
     <origin xyz="0 ${distance_between_wheels/2} ${wheel_drop_z  + base_link_z_offset}" rpy="${-pi/2} 0 0"/>
   </xacro:wheel_with_wheeldrop>
-  <xacro:wheel_with_wheeldrop name="right" namespace="$(arg namespace)">
+  <xacro:wheel_with_wheeldrop name="right" gazebo="$(arg gazebo)" namespace="$(arg namespace)">
     <origin xyz="0 ${-distance_between_wheels/2} ${wheel_drop_z  + base_link_z_offset}" rpy="${-pi/2} 0 0"/>
   </xacro:wheel_with_wheeldrop>
@@ -83,5 +86,5 @@
   </xacro:caster>
   <!-- IMU -->
-  <xacro:imu_sensor namespace="$(arg namespace)">
+  <xacro:imu_sensor gazebo="$(arg gazebo)" namespace="$(arg namespace)">
     <origin xyz="0.050613 0.043673 ${0.0202 + base_link_z_offset}"/>
   </xacro:imu_sensor>
@@ -99,5 +102,5 @@
   </gazebo>
   <!-- Mouse -->
-  <xacro:optical_mouse namespace="$(arg namespace)">
+  <xacro:optical_mouse gazebo="$(arg gazebo)" namespace="$(arg namespace)">
     <origin xyz="0.1015 0.087 ${-0.055 + base_link_z_offset}" rpy="0 0 ${-pi/4}"/>
   </xacro:optical_mouse>
@@ -112,17 +115,17 @@
   <xacro:property name="cliff_back_pitch" value="${80*deg2rad}"/>
   <xacro:property name="cliff_back_yaw" value="${167.4*deg2rad}"/>
-  <xacro:cliff_sensor name="side_left" visualize="$(arg visualize_rays)" namespace="$(arg namespace)">
+  <xacro:cliff_sensor name="side_left" gazebo="$(arg gazebo)" visualize="$(arg visualize_rays)" namespace="$(arg namespace)">
     <origin xyz="${cliff_back_x} ${cliff_back_y} ${cliff_z + base_link_z_offset}"
             rpy="0 ${cliff_back_pitch} ${cliff_back_yaw}"/>
   </xacro:cliff_sensor>
-  <xacro:cliff_sensor name="side_right" visualize="$(arg visualize_rays)" namespace="$(arg namespace)">
+  <xacro:cliff_sensor name="side_right" gazebo="$(arg gazebo)" visualize="$(arg visualize_rays)" namespace="$(arg namespace)">
     <origin xyz="${cliff_back_x} ${- cliff_back_y} ${cliff_z + base_link_z_offset}"
             rpy="0 ${cliff_back_pitch} ${- cliff_back_yaw}"/>
   </xacro:cliff_sensor>
-  <xacro:cliff_sensor name="front_left" visualize="$(arg visualize_rays)" namespace="$(arg namespace)">
+  <xacro:cliff_sensor name="front_left" gazebo="$(arg gazebo)" visualize="$(arg visualize_rays)" namespace="$(arg namespace)">
     <origin xyz="${cliff_center_x} ${cliff_center_y} ${cliff_z + base_link_z_offset}"
             rpy="0 ${cliff_center_pitch} ${cliff_center_yaw}"/>
   </xacro:cliff_sensor>
-  <xacro:cliff_sensor name="front_right" visualize="$(arg visualize_rays)" namespace="$(arg namespace)">
+  <xacro:cliff_sensor name="front_right" gazebo="$(arg gazebo)" visualize="$(arg visualize_rays)" namespace="$(arg namespace)">
     <origin xyz="${cliff_center_x} ${- cliff_center_y} ${cliff_z + base_link_z_offset}"
             rpy="0 ${cliff_center_pitch} ${- cliff_center_yaw}"/>
@@ -143,23 +146,23 @@
   side_left                                                   right
   -->
-  <xacro:ir_intensity name="front_center_left" namespace="$(arg namespace)">
+  <xacro:ir_intensity name="front_center_left" gazebo="$(arg gazebo)" namespace="$(arg namespace)">
     <origin xyz="0.1540 0 ${ir_intensity_z_pos + base_link_z_offset}"/>
   </xacro:ir_intensity>
-  <xacro:ir_intensity name="front_center_right" namespace="$(arg namespace)">
+  <xacro:ir_intensity name="front_center_right" gazebo="$(arg gazebo)" namespace="$(arg namespace)">
     <origin xyz="0.1396 -0.0651 ${ir_intensity_z_pos + base_link_z_offset}" rpy="0 0 -0.436"/>
   </xacro:ir_intensity>
-  <xacro:ir_intensity name="front_left" namespace="$(arg namespace)">
+  <xacro:ir_intensity name="front_left" gazebo="$(arg gazebo)" namespace="$(arg namespace)">
     <origin xyz="0.1396 0.0651 ${ir_intensity_z_pos + base_link_z_offset}" rpy="0 0 0.436"/>
   </xacro:ir_intensity>
-  <xacro:ir_intensity name="front_right" namespace="$(arg namespace)">
+  <xacro:ir_intensity name="front_right" gazebo="$(arg gazebo)" namespace="$(arg namespace)">
     <origin xyz="0.0990 -0.1180 ${ir_intensity_z_pos + base_link_z_offset}" rpy="0 0 -0.873"/>
   </xacro:ir_intensity>
-  <xacro:ir_intensity name="left" namespace="$(arg namespace)">
+  <xacro:ir_intensity name="left" gazebo="$(arg gazebo)" namespace="$(arg namespace)">
     <origin xyz="0.0990 0.1180 ${ir_intensity_z_pos + base_link_z_offset}" rpy="0 0 0.873"/>
   </xacro:ir_intensity>
-  <xacro:ir_intensity name="right" namespace="$(arg namespace)">
+  <xacro:ir_intensity name="right" gazebo="$(arg gazebo)" namespace="$(arg namespace)">
     <origin xyz="0.0399 -0.1488 ${ir_intensity_z_pos + base_link_z_offset}" rpy="0 0 -1.309"/>
   </xacro:ir_intensity>
-  <xacro:ir_intensity name="side_left" namespace="$(arg namespace)">
+  <xacro:ir_intensity name="side_left" gazebo="$(arg gazebo)" namespace="$(arg namespace)">
     <origin xyz="0.0399 0.1488 ${ir_intensity_z_pos + base_link_z_offset}" rpy="0 0 1.309"/>
   </xacro:ir_intensity>
@@ -180,5 +183,5 @@
   <xacro:property name="ir_omni_fov_rad" value="${220.0*deg2rad}"/>
   <xacro:property name="ir_front_facing_fov_rad" value="${pi/2}"/>
-  <xacro:ir_opcode_receivers namespace="$(arg namespace)"
+  <xacro:ir_opcode_receivers gazebo="$(arg gazebo)" namespace="$(arg namespace)"
     robot_model_name="${robot_model_name}" dock_model_name="${dock_model_name}"
     emitter_link_name="${emitter_link_name}" sensor_0_range="0.01" sensor_0_fov="${ir_omni_fov_rad}"

File: irobot_create_common/irobot_create_description/urdf/dock/ir_emitter.urdf.xacro (robot description, xacro)
@@ -6,5 +6,6 @@
                                          update_rate:=1.0
                                          min_range:=${7*cm2m}
-                                         visualize:=false" >
+                                         visualize:=false
+                                         gazebo:=ignition" >
     <!-- Physical link properties -->
     <xacro:property name="mass" value="0.15" />
@@ -24,5 +25,5 @@
     <xacro:if value="${visualize}">
       <gazebo reference="${name}_link">
-        <xacro:ray_sensor sensor_name="${name}"
+        <xacro:ray_sensor sensor_name="${name}" gazebo="${gazebo}"
                       update_rate="${update_rate}" visualize="${visualize}"
                       h_samples="50" h_res="1.0" h_min_angle="-${aperture/2}" h_max_angle="${aperture/2}"

File: irobot_create_common/irobot_create_description/urdf/dock/standard_dock.urdf.xacro (robot description, xacro)
@@ -3,4 +3,6 @@
   <xacro:include filename="$(find irobot_create_description)/urdf/common_properties.urdf.xacro"/>
   <xacro:include filename="$(find irobot_create_description)/urdf/dock/ir_emitter.urdf.xacro"/>
+  <!-- Gazebo version (kept for legacy reasons) -->
+  <xacro:arg name="gazebo"         default="ignition" />
   <xacro:arg name="namespace"      default="" />
   <xacro:property name="z_offset"  value="${4.6*mm2m}"/>
@@ -35,4 +37,5 @@
   <xacro:ir_emitter name="${green_buoy_name}"
                     parent="${link_name}"
+                    gazebo="$(arg gazebo)"
                     aperture="${buoy_lateral_aperture}"
                     max_range="1.0"
@@ -44,4 +47,5 @@
   <xacro:ir_emitter name="${red_buoy_name}"
                     parent="${link_name}"
+                    gazebo="$(arg gazebo)"
                     aperture="${buoy_lateral_aperture}"
                     max_range="1.0"
@@ -53,4 +57,5 @@
   <xacro:ir_emitter name="${yellow_buoy_name}"
                     parent="${link_name}"
+                    gazebo="$(arg gazebo)"
                     aperture="${10*deg2rad}"
                     max_range="1.0"
@@ -61,4 +66,5 @@
   <xacro:ir_emitter name="${halo_name}"
                     parent="${link_name}"
+                    gazebo="$(arg gazebo)"
                     aperture="360"
                     max_range="0.6096"

File: irobot_create_common/irobot_create_description/urdf/sensors/cliff_sensor.urdf.xacro (robot description, xacro)
@@ -2,5 +2,5 @@
 <robot xmlns:xacro="http://ros.org/wiki/xacro">
 <xacro:macro name="cliff_sensor" params="name namespace parent:=base_link
-                                         visualize:=false *origin">
+                                         visualize:=false gazebo:=ignition *origin">
   <!-- Sensor settings -->
   <xacro:property name="update_rate"         value="62"/>
@@ -21,5 +21,5 @@
   </link>
   <gazebo reference="${sensor_name}">
-    <xacro:ray_sensor sensor_name="${sensor_name}"
+    <xacro:ray_sensor sensor_name="${sensor_name}" gazebo="${gazebo}"
                       update_rate="${update_rate}" visualize="${visualize}"
                       h_samples="${samples}" h_res="1.0" h_min_angle="-${fov_rad/2}" h_max_angle="${fov_rad/2}"

File: irobot_create_common/irobot_create_description/urdf/sensors/imu.urdf.xacro (robot description, xacro)
@@ -1,5 +1,5 @@
 <?xml version="1.0"?>
 <robot xmlns:xacro="http://ros.org/wiki/xacro">
-<xacro:macro name="imu_sensor" params="name:=imu namespace parent:=base_link update_rate:=62 *origin">
+<xacro:macro name="imu_sensor" params="name:=imu namespace parent:=base_link update_rate:=62 gazebo:=ignition *origin">
   <joint name="${name}_joint" type="fixed">
     <xacro:insert_block name="origin"/>

File: irobot_create_common/irobot_create_description/urdf/sensors/ir_intensity.urdf.xacro (robot description, xacro)
@@ -6,5 +6,5 @@
                        update_rate:=62.0 fov:=${10*deg2rad}
                        min_range:=${25*mm2m} max_range:=${200*mm2m}
-                       visualize:=false *origin" >
+                       visualize:=false gazebo:=ignition *origin" >
     <xacro:property name="link_name" value="ir_intensity_${name}"/>
     <joint name="${link_name}_joint" type="fixed">
@@ -20,5 +20,5 @@
     </gazebo>
     <gazebo reference="${link_name}">
-      <xacro:ray_sensor sensor_name="${link_name}"
+      <xacro:ray_sensor sensor_name="${link_name}" gazebo="${gazebo}"
                       update_rate="${update_rate}" visualize="${visualize}"
                       h_samples="5" h_res="1.0" h_min_angle="-${fov/2}" h_max_angle="${fov/2}"

File: irobot_create_common/irobot_create_description/urdf/sensors/ir_opcode_receivers.urdf.xacro (robot description, xacro)
@@ -15,4 +15,5 @@
                                                   update_rate:=62
                                                   visualize:=false
+                                                  gazebo:=ignition
                                                   *origin" >
     <xacro:property name="joint_name" value="${name}_joint" />
@@ -31,5 +32,5 @@
       <!-- Sensor 0 visualization -->
       <gazebo reference="${receiver_link_name}">
-        <xacro:ray_sensor sensor_name="sensor_0"
+        <xacro:ray_sensor sensor_name="sensor_0" gazebo="${gazebo}"
                       update_rate="1" visualize="${visualize}"
                       h_samples="${samples}" h_res="1.0" h_min_angle="-${sensor_0_fov/2}" h_max_angle="${sensor_0_fov/2}"
@@ -38,5 +39,5 @@
       <!-- Sensor 1 visualization -->
       <gazebo reference="${receiver_link_name}">
-        <xacro:ray_sensor sensor_name="sensor_1"
+        <xacro:ray_sensor sensor_name="sensor_1" gazebo="${gazebo}"
                       update_rate="1" visualize="${visualize}"
                       h_samples="${samples}" h_res="1.0" h_min_angle="-${sensor_1_fov/2}" h_max_angle="${sensor_1_fov/2}"

File: irobot_create_common/irobot_create_description/urdf/sensors/optical_mouse.urdf.xacro (robot description, xacro)
@@ -1,5 +1,5 @@
 <?xml version="1.0"?>
 <robot xmlns:xacro="http://ros.org/wiki/xacro">
-  <xacro:macro name="optical_mouse" params="name:=mouse namespace parent_link:=base_link update_rate:=62 *origin" >
+  <xacro:macro name="optical_mouse" params="name:=mouse namespace parent_link:=base_link update_rate:=62 gazebo:=ignition *origin" >
     <joint name="${name}_joint" type="fixed">
       <xacro:insert_block name="origin"/>

File: irobot_create_common/irobot_create_description/urdf/wheel.urdf.xacro (robot description, xacro)
@@ -1,5 +1,5 @@
 <?xml version="1.0"?>
 <robot xmlns:xacro="http://ros.org/wiki/xacro">
-<xacro:macro name="wheel" params="name parent_link *origin">
+<xacro:macro name="wheel" params="name parent_link gazebo:=ignition *origin">
   <xacro:property name="mass"   value="0.2" />
   <xacro:property name="radius" value="${3.575*cm2m}" />

File: irobot_create_common/irobot_create_description/urdf/wheel_drop.urdf.xacro (robot description, xacro)
@@ -1,5 +1,5 @@
 <?xml version="1.0"?>
 <robot xmlns:xacro="http://ros.org/wiki/xacro">
-<xacro:macro name="wheel_drop" params="name parent_link namespace *origin" >
+<xacro:macro name="wheel_drop" params="name parent_link namespace gazebo:=ignition *origin" >
   <xacro:include filename="$(find irobot_create_description)/urdf/common_properties.urdf.xacro"/>
   <xacro:property name="detection_threshold" value="${3*cm2m}"/>

File: irobot_create_common/irobot_create_description/urdf/wheel_with_wheeldrop.urdf.xacro (robot description, xacro)
@@ -1,13 +1,13 @@
 <?xml version="1.0"?>
 <robot xmlns:xacro="http://ros.org/wiki/xacro">
-<xacro:macro name="wheel_with_wheeldrop" params="name namespace parent_link:=base_link *origin">
+<xacro:macro name="wheel_with_wheeldrop" params="name namespace parent_link:=base_link gazebo:=ignition *origin">
   <xacro:include filename="$(find irobot_create_description)/urdf/wheel.urdf.xacro" />
   <xacro:include filename="$(find irobot_create_description)/urdf/wheel_drop.urdf.xacro" />
   <!-- Wheel Drop definition -->
-  <xacro:wheel_drop name="${name}" parent_link="${parent_link}" namespace="${namespace}">
+  <xacro:wheel_drop name="${name}" gazebo="${gazebo}" parent_link="${parent_link}" namespace="${namespace}">
     <xacro:insert_block name="origin"/>
   </xacro:wheel_drop>
   <!-- Wheel definition -->
-  <xacro:wheel name="${name}" parent_link="wheel_drop_${name}">
+  <xacro:wheel name="${name}" gazebo="${gazebo}" parent_link="wheel_drop_${name}">
     <origin xyz="0 0 0" rpy="0 0 0"/>
   </xacro:wheel>
